File: KicadJE_ADSR_Mega32/KicadJE_ADSR_Mega32.kicad_pcb (KiCad board)
At the start: 2 copper layers, 100 x 100 mm, 134 parts, among them J101 ADSR1, J102 ADSR2, J103 ADSR1, J104 ADSR2, J105 ADSR1-G8, J106 ADSR2-G8, J107 ADSR4-G8, J108 ADSR3-G8, J201 AVR-ISP-6, J202 UART, J301 In, J302 +5V reg/doepfer, J303 Out, J304 CV_time, J305 CV doepfer, P101 Doepfer_Power_16pin, P302 Doepfer_Power_16pin, Q301 BC337, Q302 PZT2222A, U201 ATmega32A-AU, U301 L78L05_TO92, U302 PT2399, Y201 16MHz

Commit message: Update KicadJE_ADSR_Mega32.kicad_pcb
Parts:
- C209, C210: moved to F.Cu
- moved R101 18.9 mm to (65.5, 101.5), turned to 180 degrees
- moved J202 18.3 mm to (87.0, 111.0), turned to 0 degrees
- moved R102 17.9 mm to (65.5, 99.8), turned to 180 degrees
- moved Y201 8.84 mm to (86.0, 93.0), turned to 90 degrees
- moved R202 5.62 mm to (78.2, 94.5)
- moved C211 5.48 mm to (81.5, 88.8)
- moved R204 4.95 mm to (72.5, 98.0), turned to 270 degrees
- moved C210 4.76 mm to (84.2, 88.2), turned to 270 degrees
- moved C209 4.12 mm to (84.2, 92.0), turned to 90 degrees
- moved D201 1.54 mm to (78.2, 96.2), turned to 0 degrees
- moved C201 0.25 mm to (84.0, 97.8)
Routing:
- net Net-(C211-Pad2): track 17.3 -> 0.00 mm, vias 1 -> 0
- net Net-(C210-Pad1): track 7.23 -> 17.2 mm
- net 9_Tx: track 10.7 -> 1.67 mm
- net Net-(C209-Pad1): track 3.95 -> 12.7 mm
- net +5V: track 64.9 -> 58.5 mm, vias 2 -> 1
- net GND: track 71.2 -> 65.4 mm, vias 5 -> 3
- net reset: track 9.12 -> 3.81 mm, vias 1 -> 0
- net 8_Rx: track 5.97 -> 1.98 mm
